Commit message: teacher train for xbot

File: human2humanoid/resources/robots/rel2/urdf/rel2.urdf (robot description, URDF)
Before this commit: robot Xbot-L, 87 links, 86 joints
Joints:
- joint left_shoulder_roll_joint: limit lower=-2.79 upper=0.37 effort=80 velocity=7 -> lower=-2.79 upper=2.79 effort=80 velocity=7
- joint right_shoulder_roll_joint: limit lower=-0.37 upper=2.79 effort=80 velocity=7 -> lower=-2.79 upper=2.79 effort=80 velocity=7

Commit message: student policy

File: human2humanoid/resources/robots/rel2/urdf/rel2.urdf (robot description, URDF)
Before this commit: robot Xbot-L, 87 links, 86 joints
Joints:
- joint left_arm_yaw_joint: type revolute -> fixed
- joint left_wrist_yaw_joint: type revolute -> fixed
- joint right_arm_yaw_joint: type revolute -> fixed
- joint right_wrist_yaw_joint: type revolute -> fixed
